File: circuit/fortuna_terminal/fortuna_terminal.kicad_sch (KiCad schematic)
At the start: 9 parts

Commit message: WIP
Parts:
- added R?: 10K, symbol Device:R
Connections:
- net +5V: now also R?.1
- net SUSPEND_5V: now also R?.2
Changed lines of the file:
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@@
+    (stroke (width 0) (type default) (color 0 0 0 0))
+  )
+  (wire (pts (xy 189.23 52.07) (xy 189.23 80.01))
     (stroke (width 0) (type default) (color 0 0 0 0))
   )
@@
   )
   (wire (pts (xy 148.59 82.55) (xy 148.59 104.14))
+    (stroke (width 0) (type default) (color 0 0 0 0))
+  )
+  (wire (pts (xy 189.23 38.1) (xy 189.23 44.45))
     (stroke (width 0) (type default) (color 0 0 0 0))
   )
@@
     (pin "9")
   )
+  (symbol (lib_id "power:+5V") (at 189.23 38.1 0) (unit 1)
+    (in_bom yes) (on_board yes) (fields_autoplaced)
+    (property "Reference" "#PWR?" (id 0) (at 189.23 41.91 0)
+      (effects (font (size 1.27 1.27)) hide)
+    )
+    (property "Value" "+5V" (id 1) (at 189.23 33.02 0))
+    (property "Footprint" "" (id 2) (at 189.23 38.1 0)
+      (effects (font (size 1.27 1.27)) hide)
+    )
+    (property "Datasheet" "" (id 3) (at 189.23 38.1 0)
+      (effects (font (size 1.27 1.27)) hide)
+    )
+    (pin "1")
+  )
   (symbol (lib_id "power:GND") (at 74.93 116.84 0) (unit 1)
     (in_bom yes) (on_board yes) (fields_autoplaced)
@@
     (pin "9")
   )
+  (symbol (lib_id "Device:R") (at 189.23 48.26 0) (unit 1)
+    (in_bom yes) (on_board yes)
+    (property "Reference" "R?" (id 0) (at 184.15 46.99 0)
+      (effects (font (size 1.27 1.27)) (justify left))
+    )
+    (property "Value" "10K" (id 1) (at 182.88 49.53 0)
+      (effects (font (size 1.27 1.27)) (justify left))
+    )
+    (property "Footprint" "" (id 2) (at 187.452 48.26 90)
+      (effects (font (size 1.27 1.27)) hide)
+    )
+    (property "Datasheet" "~" (id 3) (at 189.23 48.26 0)
+      (effects (font (size 1.27 1.27)) hide)
+    )
+    (pin "1")
+    (pin "2")
+  )
   (symbol (lib_id "power:+3.3V") (at 226.06 92.71 0) (unit 1)
     (in_bom yes) (on_board yes)
@@
       (reference "#PWR?") (unit 1) (value "GND") (footprint "")
     )
+    (path "/c77b47f1-b1eb-46f3-be61-d48d6624f9fe"
+      (reference "#PWR?") (unit 1) (value "+5V") (footprint "")
+    )
     (path "/c781f31f-b35e-447d-92a3-bc27c0eb4452"
       (reference "#PWR?") (unit 1) (value "GND") (footprint "")
@@
       (reference "R?") (unit 1) (value "10K") (footprint "")
     )
+    (path "/d02c9c1c-c39f-4492-9499-64b35ecc5703"
+      (reference "R?") (unit 1) (value "10K") (footprint "")
+    )

Commit message: WIP
Connections:
- net REMOTE: no longer J?.3 (Pin_3), J?.3 (Pin_3), J?.7 (GCLK0/GPIO4)
- net CMD_5V: now reaches U?.10 (B4)
- net CMD_5V: now also J?.3 (Pin_3), J?.3 (Pin_3)
- net CMD: now reaches U?.5 (A4)
Other:
- note added: "VNSYC (OUT) - notifies the master when a frame has finished RST (IN/OUT) - resets the master SUSPEND (IN) - suspend communication while line is down CMD (IN) - when down, master is sending commands (when using Fortuna+ANSI) MOSI, MISO, SCK - SPI communication RX, TX - serial communication SDA, SCL - I²C communication"
Changed lines of the file:
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@@
   (junction (at 144.78 87.63) (diameter 0) (color 0 0 0 0)
   )
-  (junction (at 137.16 85.09) (diameter 0) (color 0 0 0 0)
-  )
   (junction (at 144.78 63.5) (diameter 0) (color 0 0 0 0)
   )
@@
   (junction (at 140.97 90.17) (diameter 0) (color 0 0 0 0)
   )
+  (junction (at 137.16 109.22) (diameter 0) (color 0 0 0 0)
+  )
   (wire (pts (xy 105.41 91.44) (xy 115.57 91.44))
     (stroke (width 0) (type default) (color 0 0 0 0))
@@
     (stroke (width 0) (type default) (color 0 0 0 0))
   )
+  (wire (pts (xy 137.16 109.22) (xy 160.02 109.22))
+    (stroke (width 0) (type default) (color 0 0 0 0))
+  )
   (wire (pts (xy 57.15 63.5) (xy 64.77 63.5))
     (stroke (width 0) (type default) (color 0 0 0 0))
@@
     (stroke (width 0) (type default) (color 0 0 0 0))
   )
-  (wire (pts (xy 137.16 76.2) (xy 137.16 85.09))
-    (stroke (width 0) (type default) (color 0 0 0 0))
-  )
   (wire (pts (xy 144.78 63.5) (xy 144.78 87.63))
     (stroke (width 0) (type default) (color 0 0 0 0))
@@
     (stroke (width 0) (type default) (color 0 0 0 0))
   )
+  (wire (pts (xy 218.44 116.84) (xy 137.16 116.84))
+    (stroke (width 0) (type default) (color 0 0 0 0))
+  )
   (wire (pts (xy 213.36 71.12) (xy 213.36 82.55))
     (stroke (width 0) (type default) (color 0 0 0 0))
@@
     (stroke (width 0) (type default) (color 0 0 0 0))
   )
-  (wire (pts (xy 137.16 109.22) (xy 137.16 85.09))
-    (stroke (width 0) (type default) (color 0 0 0 0))
-  )
   (wire (pts (xy 148.59 55.88) (xy 148.59 58.42))
     (stroke (width 0) (type default) (color 0 0 0 0))
@@
     (stroke (width 0) (type default) (color 0 0 0 0))
   )
+  (wire (pts (xy 137.16 85.09) (xy 137.16 109.22))
+    (stroke (width 0) (type default) (color 0 0 0 0))
+  )
   (wire (pts (xy 180.34 60.96) (xy 180.34 71.12))
     (stroke (width 0) (type default) (color 0 0 0 0))
@@
     (stroke (width 0) (type default) (color 0 0 0 0))
   )
+  (wire (pts (xy 160.02 85.09) (xy 137.16 85.09))
+    (stroke (width 0) (type default) (color 0 0 0 0))
+  )
   (wire (pts (xy 144.78 111.76) (xy 144.78 127))
     (stroke (width 0) (type default) (color 0 0 0 0))
@@
     (stroke (width 0) (type default) (color 0 0 0 0))
   )
-  (wire (pts (xy 160.02 109.22) (xy 137.16 109.22))
-    (stroke (width 0) (type default) (color 0 0 0 0))
-  )
   (wire (pts (xy 226.06 91.44) (xy 226.06 92.71))
     (stroke (width 0) (type default) (color 0 0 0 0))
@@
     (stroke (width 0) (type default) (color 0 0 0 0))
   )
+  (wire (pts (xy 137.16 116.84) (xy 137.16 109.22))
+    (stroke (width 0) (type default) (color 0 0 0 0))
+  )
   (wire (pts (xy 189.23 80.01) (xy 210.82 80.01))
     (stroke (width 0) (type default) (color 0 0 0 0))
@@
     (stroke (width 0) (type default) (color 0 0 0 0))
   )
+  (wire (pts (xy 238.76 116.84) (xy 250.19 116.84))
+    (stroke (width 0) (type default) (color 0 0 0 0))
+  )
   (wire (pts (xy 105.41 96.52) (xy 121.92 96.52))
     (stroke (width 0) (type default) (color 0 0 0 0))
@@
     (stroke (width 0) (type default) (color 0 0 0 0))
   )
-  (wire (pts (xy 105.41 76.2) (xy 137.16 76.2))
-    (stroke (width 0) (type default) (color 0 0 0 0))
-  )
   (wire (pts (xy 180.34 71.12) (xy 121.92 71.12))
     (stroke (width 0) (type default) (color 0 0 0 0))
   )
-  (wire (pts (xy 137.16 85.09) (xy 160.02 85.09))
-    (stroke (width 0) (type default) (color 0 0 0 0))
-  )
   (wire (pts (xy 144.78 127) (xy 52.07 127))
     (stroke (width 0) (type default) (color 0 0 0 0))
@@
     (stroke (width 0) (type default) (color 0 0 0 0))
   )
+  (text "VNSYC (OUT)  - notifies the master when a frame has finished\nRST (IN/OUT) - resets the master\nSUSPEND (IN) - suspend communication while line is down\nCMD (IN)     - when down, master is sending commands (when using Fortuna+ANSI)\n\nMOSI, MISO, SCK - SPI communication\nRX, TX          - serial communication\nSDA, SCL        - I²C communication"
+    (at 62.23 156.21 0)
+    (effects (font (size 1.27 1.27)) (justify left bottom))
+  )
   (label "SCK" (at 115.57 96.52 180)
     (effects (font (size 1.27 1.27)) (justify right bottom))
@@
     (effects (font (size 1.27 1.27)) (justify left bottom))
   )
-  (label "REMOTE" (at 152.4 109.22 0)
+  (label "CMD_5V" (at 152.4 109.22 0)
     (effects (font (size 1.27 1.27)) (justify left bottom))
   )
@@
     (effects (font (size 1.27 1.27)) (justify left bottom))
   )
+  (label "TX_5V" (at 213.36 71.12 270)
+    (effects (font (size 1.27 1.27)) (justify right bottom))
+  )
   (label "SCL_5V" (at 182.88 109.22 180)
     (effects (font (size 1.27 1.27)) (justify right bottom))
@@
     (effects (font (size 1.27 1.27)) (justify left bottom))
   )
+  (label "CMD_5V" (at 209.55 116.84 0)
+    (effects (font (size 1.27 1.27)) (justify left bottom))
+  )
   (label "SCL" (at 250.19 111.76 180)
     (effects (font (size 1.27 1.27)) (justify right bottom))
@@
     (effects (font (size 1.27 1.27)) (justify right bottom))
   )
+  (label "RX_5V" (at 213.36 101.6 90)
+    (effects (font (size 1.27 1.27)) (justify left bottom))
+  )
   (label "RX" (at 250.19 101.6 180)
     (effects (font (size 1.27 1.27)) (justify right bottom))
@@
     (effects (font (size 1.27 1.27)) (justify left bottom))
   )
-  (label "REMOTE" (at 152.4 85.09 0)
+  (label "CMD_5V" (at 152.4 85.09 0)
     (effects (font (size 1.27 1.27)) (justify left bottom))
   )
@@
     (effects (font (size 1.27 1.27)) (justify right bottom))
   )
+  (label "SUSPEND_5V" (at 210.82 66.04 270)
+    (effects (font (size 1.27 1.27)) (justify right bottom))
+  )
   (label "MOSI" (at 152.4 60.96 0)
     (effects (font (size 1.27 1.27)) (justify left bottom))
@@
     (effects (font (size 1.27 1.27)) (justify right bottom))
   )
+  (label "CMD" (at 250.19 116.84 180)
+    (effects (font (size 1.27 1.27)) (justify right bottom))
+  )

Commit message: WIP
Parts:
- removed J?: Raspberry_Pi_2_3, symbol Connector:Raspberry_Pi_2_3
- removed SW?: USR, symbol Switch:SW_Push
- added D?: LED, symbol Device:LED
- added J?: Raspberry Pi Zero, symbol Connector_Generic:Conn_02x20_Odd_Even
- added R?: 220, symbol Device:R
- added SW?: USR, symbol Switch:SW_Push
Connections:
- net +3.3V: now also J?.1 (Pin_1)
- net +5V: now also J?.2 (Pin_2), R?.1
- net GND: now also D?.2 (A), J?.6 (Pin_6), J?.9 (Pin_9), SW?.1
- net MISO: now also J?.21 (Pin_21)
- net MOSI: now also J?.19 (Pin_19)
- net RST: now also J?.18 (Pin_18)
- net RX: now also J?.10 (Pin_10)
- net SCK: now also J?.23 (Pin_23)
- net SCL: now also J?.5 (Pin_5)
- net SDA: now also J?.3 (Pin_3)
- net SUSPEND: now also J?.31 (Pin_31)
- net TX: now also J?.8 (Pin_8)
- net VSYNC: now also J?.29 (Pin_29)
- new net: J?.11 (Pin_11), SW?.2
- new net: D?.1 (K), R?.2
- no-connect marks 0 -> 25
Other:
- note added: "Rest of Pi is here, seen from above"
- moved on the sheet: J?, R?, SW?, U?

Commit message: WIP
Parts:
- added C?: 10uF, symbol Device:C_Small
- added J?: ATMEGA328, symbol Connector_Generic:Conn_02x14_Counter_Clockwise
Connections:
- net +5V: now also C?.1, J?.7 (Pin_7)
- net CMD_5V: now also J?.26 (Pin_26)
- net CS_5V: now also J?.16 (Pin_16)
- net GND: now also C?.2, J?.8 (Pin_8)
- net MISO_5V: now also J?.18 (Pin_18)
- net MOSI: now also J?.17 (Pin_17)
- net RST: now also J?.1 (Pin_1)
- net RX_5V: now also J?.3 (Pin_3)
- net SCK: now also J?.19 (Pin_19)
- net SCL_5V: now also J?.28 (Pin_28)
- net SDA_5V: now also J?.27 (Pin_27)
- net SUSPEND_5V: now also J?.25 (Pin_25)
- net TX_5V: now also J?.2 (Pin_2)
Other:
- note added: "TEST CIRCUIT"
- moved on the sheet: D?, J?, R?, SW?, U?

Commit message: WIP
Connections:
- net CS: now also J?.16 (Pin_16)
- net SUSPEND: now also J?.15 (Pin_15); no longer J?.31 (Pin_31)
- net VSYNC: now also J?.13 (Pin_13); no longer J?.29 (Pin_29)
- no-connect marks 25 -> 24
Other:
- moved on the sheet: SW?
Changed lines of the file:
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@@
   )
   (no_connect (at 113.03 43.18))
-  (no_connect (at 113.03 58.42))
   (no_connect (at 113.03 55.88))
   (no_connect (at 113.03 53.34))
   (no_connect (at 100.33 48.26))
+  (no_connect (at 100.33 76.2))
+  (no_connect (at 100.33 78.74))
   (no_connect (at 113.03 68.58))
   (no_connect (at 113.03 66.04))
   (no_connect (at 113.03 63.5))
   (no_connect (at 100.33 60.96))
-  (no_connect (at 100.33 58.42))
-  (no_connect (at 100.33 55.88))
   (no_connect (at 100.33 86.36))
   (no_connect (at 100.33 81.28))
@@
   (no_connect (at 113.03 81.28))
   (no_connect (at 100.33 88.9))
+  (wire (pts (xy 113.03 58.42) (xy 123.19 58.42))
+    (stroke (width 0) (type default) (color 0 0 0 0))
+  )
   (wire (pts (xy 160.02 43.18) (xy 163.83 43.18))
     (stroke (width 0) (type default) (color 0 0 0 0))
@@
     (stroke (width 0) (type default) (color 0 0 0 0))
   )
+  (wire (pts (xy 90.17 58.42) (xy 100.33 58.42))
+    (stroke (width 0) (type default) (color 0 0 0 0))
+  )
   (wire (pts (xy 113.03 60.96) (xy 123.19 60.96))
     (stroke (width 0) (type default) (color 0 0 0 0))
@@
     (stroke (width 0) (type default) (color 0 0 0 0))
   )
-  (wire (pts (xy 91.44 53.34) (xy 100.33 53.34))
+  (wire (pts (xy 87.63 53.34) (xy 100.33 53.34))
     (stroke (width 0) (type default) (color 0 0 0 0))
   )
@@
     (stroke (width 0) (type default) (color 0 0 0 0))
   )
-  (wire (pts (xy 90.17 78.74) (xy 100.33 78.74))
-    (stroke (width 0) (type default) (color 0 0 0 0))
-  )
   (wire (pts (xy 200.66 87.63) (xy 200.66 109.22))
     (stroke (width 0) (type default) (color 0 0 0 0))
@@
     (stroke (width 0) (type default) (color 0 0 0 0))
   )
-  (wire (pts (xy 90.17 76.2) (xy 100.33 76.2))
-    (stroke (width 0) (type default) (color 0 0 0 0))
-  )
   (wire (pts (xy 187.96 58.42) (xy 195.58 58.42))
     (stroke (width 0) (type default) (color 0 0 0 0))
@@
     (stroke (width 0) (type default) (color 0 0 0 0))
   )
-  (wire (pts (xy 81.28 53.34) (xy 76.2 53.34))
+  (wire (pts (xy 77.47 53.34) (xy 76.2 53.34))
     (stroke (width 0) (type default) (color 0 0 0 0))
   )
@@
   )
   (wire (pts (xy 156.21 87.63) (xy 175.26 87.63))
+    (stroke (width 0) (type default) (color 0 0 0 0))
+  )
+  (wire (pts (xy 90.17 55.88) (xy 100.33 55.88))
     (stroke (width 0) (type default) (color 0 0 0 0))
   )
@@
     (effects (font (size 1.27 1.27)) (justify left bottom))
   )
+  (label "VSYNC" (at 90.17 55.88 0)
+    (effects (font (size 1.27 1.27)) (justify left bottom))
+  )
   (label "RST" (at 167.64 85.09 0)
     (effects (font (size 1.27 1.27)) (justify left bottom))
@@
     (effects (font (size 1.27 1.27)) (justify right bottom))
   )
-  (label "SUSPEND" (at 90.17 78.74 0)
-    (effects (font (size 1.27 1.27)) (justify left bottom))
-  )
   (label "CMD_5V" (at 224.79 114.3 0)
     (effects (font (size 1.27 1.27)) (justify left bottom))
@@
     (effects (font (size 1.27 1.27)) (justify right bottom))
   )
+  (label "SUSPEND" (at 90.17 58.42 0)
+    (effects (font (size 1.27 1.27)) (justify left bottom))
+  )
   (label "SUSPEND_5V" (at 102.87 153.67 180)
     (effects (font (size 1.27 1.27)) (justify right bottom))
@@
     (effects (font (size 1.27 1.27)) (justify right bottom))
   )
+  (label "CS" (at 123.19 58.42 180)
+    (effects (font (size 1.27 1.27)) (justify right bottom))
+  )
   (label "MOSI" (at 90.17 63.5 0)
     (effects (font (size 1.27 1.27)) (justify left bottom))
@@
   )
   (label "CMD_5V" (at 167.64 82.55 0)
-    (effects (font (size 1.27 1.27)) (justify left bottom))
-  )
-  (label "VSYNC" (at 90.17 76.2 0)
     (effects (font (size 1.27 1.27)) (justify left bottom))
   )
@@
     (pin "1")
   )
-  (symbol (lib_id "Switch:SW_Push") (at 86.36 53.34 0) (unit 1)
+  (symbol (lib_id "Switch:SW_Push") (at 82.55 53.34 0) (unit 1)
     (in_bom yes) (on_board yes)
-    (property "Reference" "SW?" (id 0) (at 87.6301 54.61 90)
+    (property "Reference" "SW?" (id 0) (at 83.8201 54.61 90)
       (effects (font (size 1.27 1.27)) (justify right))
     )
-    (property "Value" "USR" (id 1) (at 85.0901 54.61 90)
+    (property "Value" "USR" (id 1) (at 81.2801 54.61 90)
       (effects (font (size 1.27 1.27)) (justify right))
     )
-    (property "Footprint" "" (id 2) (at 86.36 48.26 0)
-      (effects (font (size 1.27 1.27)) hide)
-    )
-    (property "Datasheet" "~" (id 3) (at 86.36 48.26 0)
-      (effects (font (size 1.27 1.27)) hide)
-    )
+    (property "Footprint" "" (id 2) (at 82.55 48.26 0)
+      (effects (font (size 1.27 1.27)) hide)
+    )
+    (property "Datasheet" "~" (id 3) (at 82.55 48.26 0)
+      (effects (font (size 1.27 1.27)) hide)
+    )

Commit message: WIP
Connections:
- net RST: now also U?.10 (B4), U?.5 (A4)
- net TX: now also J?.2 (Pin_2), J?.9 (Pin_9); no longer U?.5 (A4)
- removed net TX_5V: J?.2 (Pin_2), J?.9 (Pin_9), U?.10 (B4)
Other:
- moved on the sheet: J?, R?, SW?, U?

Commit message: WIP
Parts:
- removed J?: I²C Connector, symbol Connector_Generic:Conn_02x05_Counter_Clockwise
- removed J? (x2): UART Connector, symbol Connector_Generic:Conn_02x05_Counter_Clockwise
- removed R? (x2): 10K, symbol Device:R
- removed SW?: USR, symbol Switch:SW_Push
- removed SW?: RESET, symbol Switch:SW_Push
- removed U? (x2): Level shifter, Package_SO:TSSOP-14_4.4x5mm_P0.65mm, symbol Logic_LevelTranslator:TXB0104PW
- added J?: Conn_02x08_Odd_Even, symbol Connector_Generic:Conn_02x08_Odd_Even
- added R? (x2): 10K, symbol Device:R
- added SW?: RESET, symbol Switch:SW_Push
- added U? (x2): Level shifter, Package_SO:TSSOP-14_4.4x5mm_P0.65mm, symbol Logic_LevelTranslator:TXB0104PW
Connections:
- net +3.3V: now also U?.1 (VCCA), U?.1 (VCCA)
- net +5V: now also J?.1 (Pin_1), J?.3 (Pin_3), R?.1, R?.1, U?.14 (VCCB), U?.14 (VCCB)
- net CMD: now also J?.11 (Pin_11), U?.5 (A4)
- net CMD_5V: now also J?.8 (Pin_8)
- net CS: now also U?.3 (A2)
- net CS_5V: now also J?.12 (Pin_12)
- net GND: now also J?.13 (Pin_13), J?.15 (Pin_15), SW?.1, U?.7 (GND), U?.7 (GND)
- net MISO: now also U?.4 (A3)
- net MISO_5V: now also J?.14 (Pin_14)
- net MOSI: now also J?.5 (Pin_5)
- net RST: now also J?.24 (Pin_24), U?.5 (A4); no longer J?.1 (Pin_1), J?.18 (Pin_18)
- net RX: now also U?.4 (A3)
- net RX_5V: now also J?.6 (Pin_6)
- net SCK: now also J?.7 (Pin_7)
- net SCL: now also U?.3 (A2)
- net SCL_5V: now also J?.4 (Pin_4)
- net SDA: now also U?.2 (A1)
- net SDA_5V: now also J?.2 (Pin_2)
- net SUSPEND: now also U?.2 (A1)
- net SUSPEND_5V: now also J?.10 (Pin_10), R?.2, SW?.2
- net TX: now also J?.11 (Pin_11)
- net VSYNC: now also J?.9 (Pin_9)
- new net RST_5V: J?.1 (Pin_1), J?.16 (Pin_16), R?.2
Other:
- moved on the sheet: J?

Commit message: .
Parts:
- added SW?: SW_DIP_x04, symbol Switch:SW_DIP_x04
- added SW? (x2): SW_Push, symbol Switch:SW_Push
Connections:
- net GND: now also SW?.1, SW?.1, SW?.1, SW?.2, SW?.3, SW?.4
- net at J?.11 (Pin_11): now also SW?.8
- net at J?.12 (Pin_12): now also SW?.7
- net at J?.13 (Pin_13): now also SW?.6
- net at J?.14 (Pin_14): now also SW?.5
- net at J?.4 (Pin_4): now also SW?.2
- net at J?.5 (Pin_5): now also SW?.2
Other:
- moved on the sheet: C?
