File: circuit/fortuna_terminal/fortuna_terminal.kicad_sch (KiCad schematic)
At the start: 14 parts

Commit message: .
Parts:
- added C? (x2): 33pF, symbol Device:C_Small
- added J?: Crystal, symbol Connector:Conn_01x02_Female
Connections:
- net GND: now also C?.2, C?.2
- net at J?.10 (Pin_10): now also C?.1, J?.2 (Pin_2)
- net at J?.9 (Pin_9): now also C?.1, J?.1 (Pin_1)
Other:
- moved on the sheet: C?, J?, SW?

Commit message: .
Parts:
- removed SW?: SW_Push, symbol Switch:SW_Push
Connections:
- net VSYNC: now also J?.5 (Pin_5)
Changed lines of the file:
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@@
   (junction (at 45.72 163.83) (diameter 0) (color 0 0 0 0)
-  )
-  (junction (at 58.42 151.13) (diameter 0) (color 0 0 0 0)
   )
   (junction (at 58.42 168.91) (diameter 0) (color 0 0 0 0)
@@
     (stroke (width 0) (type default) (color 0 0 0 0))
   )
+  (wire (pts (xy 72.39 151.13) (xy 80.01 151.13))
+    (stroke (width 0) (type default) (color 0 0 0 0))
+  )
   (wire (pts (xy 232.41 49.53) (xy 237.49 49.53))
     (stroke (width 0) (type default) (color 0 0 0 0))
@@
     (stroke (width 0) (type default) (color 0 0 0 0))
   )
-  (wire (pts (xy 58.42 148.59) (xy 58.42 151.13))
+  (wire (pts (xy 58.42 148.59) (xy 58.42 160.02))
     (stroke (width 0) (type default) (color 0 0 0 0))
   )
@@
     (stroke (width 0) (type default) (color 0 0 0 0))
   )
-  (wire (pts (xy 68.58 151.13) (xy 80.01 151.13))
-    (stroke (width 0) (type default) (color 0 0 0 0))
-  )
   (wire (pts (xy 269.24 54.61) (xy 269.24 57.15))
     (stroke (width 0) (type default) (color 0 0 0 0))
@@
   )
   (wire (pts (xy 213.36 59.69) (xy 213.36 66.04))
-    (stroke (width 0) (type default) (color 0 0 0 0))
-  )
-  (wire (pts (xy 58.42 151.13) (xy 58.42 160.02))
     (stroke (width 0) (type default) (color 0 0 0 0))
   )
@@
   (label "MOSI" (at 106.68 168.91 180)
     (effects (font (size 1.27 1.27)) (justify right bottom))
+  )
+  (label "VSYNC" (at 72.39 151.13 0)
+    (effects (font (size 1.27 1.27)) (justify left bottom))
   )
   (label "SCK" (at 106.68 163.83 180)
@@
     (pin "9")
   )
-  (symbol (lib_id "Switch:SW_Push") (at 63.5 151.13 0) (unit 1)
-    (in_bom yes) (on_board yes)
-    (property "Reference" "SW?" (id 0) (at 68.58 149.86 0))
-    (property "Value" "SW_Push" (id 1) (at 53.34 151.13 0))
-    (property "Footprint" "" (id 2) (at 63.5 146.05 0)
-      (effects (font (size 1.27 1.27)) hide)
-    )
-    (property "Datasheet" "~" (id 3) (at 63.5 146.05 0)
-      (effects (font (size 1.27 1.27)) hide)
-    )
-    (pin "1")
-    (pin "2")
-  )
   (symbol (lib_id "Connector_Generic:Conn_02x08_Odd_Even") (at 78.74 57.15 0) (unit 1)
     (in_bom yes) (on_board yes) (fields_autoplaced)
@@
       (reference "SW?") (unit 1) (value "SW_DIP_x04") (footprint "")
     )
-    (path "/730672a3-ddc3-4720-b8d6-97cd0b1915e9"
-      (reference "SW?") (unit 1) (value "SW_Push") (footprint "")
-    )
     (path "/b1b7a4a6-82d2-4e36-8cfe-0f1766eacbf3"

Commit message: .
Connections:
- net CS: now also J?.24 (Pin_24); no longer J?.16 (Pin_16)
- net RST: now also J?.22 (Pin_22); no longer J?.24 (Pin_24)
- no-connect marks 24 -> 23
Changed lines of the file:
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@@
   (no_connect (at 237.49 85.09))
   (no_connect (at 237.49 87.63))
-  (no_connect (at 250.19 74.93))
   (no_connect (at 250.19 72.39))
   (no_connect (at 237.49 69.85))
@@
     (stroke (width 0) (type default) (color 0 0 0 0))
   )
-  (wire (pts (xy 250.19 67.31) (xy 260.35 67.31))
-    (stroke (width 0) (type default) (color 0 0 0 0))
-  )
   (wire (pts (xy 86.36 52.07) (xy 100.33 52.07))
     (stroke (width 0) (type default) (color 0 0 0 0))
@@
   )
   (wire (pts (xy 92.71 171.45) (xy 106.68 171.45))
+    (stroke (width 0) (type default) (color 0 0 0 0))
+  )
+  (wire (pts (xy 250.19 74.93) (xy 260.35 74.93))
     (stroke (width 0) (type default) (color 0 0 0 0))
   )
@@
     (effects (font (size 1.27 1.27)) (justify right bottom))
   )
-  (label "RST" (at 260.35 77.47 180)
-    (effects (font (size 1.27 1.27)) (justify right bottom))
-  )
-  (label "CS" (at 260.35 67.31 180)
-    (effects (font (size 1.27 1.27)) (justify right bottom))
-  )
+  (label "CS" (at 260.35 77.47 180)
+    (effects (font (size 1.27 1.27)) (justify right bottom))
+  )
+  (label "RST" (at 260.35 74.93 180)
+    (effects (font (size 1.27 1.27)) (justify right bottom))
+  )
